File: Hardware/GC_Video_Adapter.kicad_pcb (KiCad board)
At the start: 4 copper layers, 40 x 58.7 mm, 78 parts, among them J1 GC_DVOUT, J2 Conn_01x08, J3 Conn_01x02, J4 Conn_01x02, J5 Conn_01x02, J6 AudioJack3, SW1 SW_DIP_x01, U1 LCMXO2-640-100TQFP, U2 ADV7125, U3 PCM5102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

Commit message: Upgraded from Kicad 5 to Kicad 8.
Connections:
- net /DAC/~DACBLANK renamed /DAC/~{DACBLANK}
- net /DAC/~DACSYNC renamed /DAC/~{DACSYNC}
Other:
- net class 75Ohm removed
- net class Default removed
- net class Power removed
